Commit message: New ikfast solvers. Testing one to link6.
Old ikfast solver is in ikfast_old.cpp.
Currently testing a solver that only goes to link 6.

I suspect that the meshes in the arm will have be aligned (again)
because I might have accidentally deleted those changes.

File: cwru_abby/abby_description/urdf/abby.urdf (robot description, URDF)
Before this commit: robot abby, 38 links, 37 joints
Links:
- added link camera_depth_frame, mass 0.01
- added link camera_depth_optical_frame, mass 0.001
- added link camera_rgb_frame, mass 0.001
- added link camera_rgb_optical_frame, mass 0.001
- added link light; collision cylinder length=0.165 radius=0.075; visual cylinder length=0.165 radius=0.075
- added link tanks; collision cylinder length=0.50 radius=0.0275; visual cylinder length=0.50 radius=0.0275
Joints:
- added joint camera_depth_joint: type fixed, parent camera_link, child camera_depth_frame, origin xyz=0 0.011 0 rpy=0 0 0
- added joint camera_depth_optical_joint: type fixed, parent camera_depth_frame, child camera_depth_optical_frame, origin xyz=0 0 0 rpy=-1.570795 0 -1.570795
- added joint camera_rgb_joint: type fixed, parent camera_link, child camera_rgb_frame, origin xyz=0 -0.012 0 rpy=0 0 0
- added joint camera_rgb_optical_joint: type fixed, parent camera_rgb_frame, child camera_rgb_optical_frame, origin xyz=0 0 0 rpy=-1.570795 0 -1.570795
- added joint frame-light: type fixed, parent frame1, child light, origin xyz=0.215 -0.45 1.3 rpy=0 1.571 0
- added joint frame-tanks: type fixed, parent frame1, child tanks, origin xyz=0.16 -0.45 0.95 rpy=0 0 0
- joint frame_arm: origin xyz=0.046 -0.55 .75 rpy=3.1415926535 1.57079632679 0 -> xyz=0.04464 -0.473311 0.753907 rpy=-1.571 1.446 1.571
